Commit message: xacro

File: src/rocker_bogie/urdf/plugins.xacro (robot description, xacro)
@@ -1,6 +1,6 @@
 <?xml version="1.0" ?>
 <robot name="plugins" xmlns:xacro="http://ros.org/wiki/xacro">
-    <gazebo reference="lidar_link">
-    <material name="black"><color rgba="0.0 0.0 0.0 1.0"/></material>
+    <gazebo reference="base_scan">
+    <material>Gazebo/FlatBlack</material>
     <sensor type="ray" name="lidar_sensor">
         <origin xyz="0 0 0.2" rpy="0 0 0"/>
@@ -13,11 +13,11 @@
             <resolution>1</resolution>
             <min_angle>0</min_angle> <!-- -90 degrees -->
-            <max_angle>6.28</max_angle>  <!-- +90 degrees -->
+            <max_angle>6.28319</max_angle>  <!-- +90 degrees -->
             </horizontal>
         </scan>
         <range>
-            <min>0.2</min> <!-- Min detection distance -->
+            <min>0.15</min> <!-- Min detection distance -->
             <max>3.5</max> <!-- Max detection distance -->
-            <resolution>0.01d</resolution>
+            <resolution>0.01</resolution>
         </range>
         <noise>
@@ -29,5 +29,5 @@
         <plugin name="gazebo_ros_laser" filename="libgazebo_ros_laser.so">
         <topicName>scan</topicName>
-        <frameName>lidar_link</frameName>
+        <frameName>base_scan</frameName>
         </plugin>
     </sensor>

File: src/rocker_bogie/urdf/rocker_bogie.urdf.xacro (robot description, xacro)
@@ -1,5 +1,7 @@
 <?xml version="1.0"?>
-<robot xmlns:xacro="http://www.ros.org/wiki/xacro" name="rocker_bogie">
+<robot name="rocker_bogie_sim" xmlns:xacro="http://www.ros.org/wiki/xacro">
+  <xacro:include filename="$(find rocker_bogie)/urdf/color.xacro"/>
   <xacro:include filename="$(find rocker_bogie)/urdf/plugins.xacro"/>
+  <xacro:include filename="$(find rocker_bogie)/urdf/rocker_bogie.gazebo.xacro"/>
   <!-- Properties for reuse -->
   <xacro:property name="wheel_radius" value="0.07"/>
@@ -9,17 +11,6 @@
   <xacro:property name="blue_color" value="0 1 1 1"/>
   <xacro:property name="orange_color" value="1 0.5 0 1"/>
-<!-- Base Link at the Center of the Chassis -->
-<link name="base_link">
-  <visual>
-    <geometry>
-      <sphere radius="0.01"/>  <!-- Small sphere for visual debugging -->
-    </geometry>
-    <origin xyz="0 0 0"/>  <!-- Centered inside the chassis -->
-    <material name="gray">
-      <color rgba="0.5 0.5 0.5 1"/>
-    </material>
-  </visual>
-</link>
-<link name="lidar_link">
+<link name="base_link"></link>
+<link name="base_scan">
   <visual>
     <origin xyz="0 0 0.1" rpy="0 0 0" />
@@ -29,14 +20,14 @@
   </visual>
 </link>
-<joint name="lidar_joint" type="fixed">
+<joint name="scan_joint" type="fixed">
   <parent link="base_link"/>
-  <child link="lidar_link"/>
-  <origin xyz="0 0 0.2" rpy="0 0 0"/> <!-- Position the LiDAR slightly above the rover chassis -->
+  <child link="base_scan"/>
+  <origin xyz="0 0 0.2" rpy="0 0 0"/>
 </joint>
 <link name="base_footprint"/>
-<joint name="base_footprint_joint" type="fixed">
+<joint name="base_joint" type="fixed">
     <parent link="base_footprint"/>
     <child link="base_link"/>
-    <origin xyz="0 0 -0.05" rpy="0 0 0"/>
+    <origin xyz="0 0 0" rpy="0 0 0"/>
 </joint>
   <!-- Macro for Chassis -->
@@ -48,7 +39,5 @@
       </geometry>
       <origin xyz="0 0 0"/>
-      <material name="green">
-        <color rgba="0 1 0 1"/>
-      </material>
+      <material name="green"/>
     </visual>
     <collision>
@@ -61,5 +50,5 @@
       <mass value="5.3"/>
       <!-- <mass value="15"/> -->
-      <origin xyz="0 0 0"/>  <!-- Set CoM to the geometric center -->
+      <origin xyz="0 0 0"/>
       <inertia ixx="0.5" ixy="0" ixz="0" iyy="0.5" iyz="0" izz="0.8"/>
     </inertial>
@@ -74,7 +63,5 @@
       </geometry>
       <origin xyz="0 ${position_y} 0" rpy="1.5707 0 0"/>
-      <material name="gray">
-        <color rgba="0.5 0.5 0.5 1"/>
-      </material>
+      <material name="grey"/>
     </visual>
     <collision>
@@ -97,15 +84,15 @@
       <geometry><box size="0.32 0.024 0.024"/></geometry>
       <origin xyz="-0.147 ${position_y} 0"/>
-      <material name="blue"><color rgba="${blue_color}"/></material>
+      <material name="blue"/>
     </visual>
     <visual> <!-- Vertical Bar Collision -->
       <geometry><box size="0.024 0.024 0.186"/></geometry>
       <origin xyz="-0.294 ${position_y} -0.1"/>
-      <material name="blue"><color rgba="${blue_color}"/></material>
+      <material name="blue"/>
     </visual>
     <visual> <!-- Rotating Bar Collision -->
       <geometry><box size="0.024 0.024 0.12"/></geometry>
       <origin xyz="0.055 ${position_y} -0.055" rpy="0 -0.61 0"/>
-      <material name="blue"><color rgba="${blue_color}"/></material>
+      <material name="blue"/>
     </visual>
     <collision> <!-- Horizontal Bar Collision -->
@@ -146,7 +133,5 @@
       </geometry>
       <origin xyz="0.177 ${position_y} 0.1"/>
-      <material name="orange">
-        <color rgba="${orange_color}"/>
-      </material>
+      <material name="orange"/>
     </visual>
     <visual> <!-- Front Vertical Bar -->
@@ -155,7 +140,5 @@
       </geometry>
       <origin xyz="0.2 ${position_y} 0.01"/>
-      <material name="orange">
-        <color rgba="${orange_color}"/>
-      </material>
+      <material name="orange"/>
     </visual>
     <visual> <!-- Back Rotating Bar -->
@@ -164,7 +147,5 @@
       </geometry>
       <origin xyz="0.01 ${position_y} 0.01" rpy="0 0.96 0"/>
-      <material name="orange">
-        <color rgba="${orange_color}"/>
-      </material>
+      <material name="orange"/>
     </visual>
     <collision> <!-- Horizontal Bar Collision -->
@@ -224,9 +205,4 @@
     <limit lower="-0.26" upper="0.26" velocity="100" effort="100"/>
     <dynamics damping="0.5" spring_stiffness="50"/>
-    <gazebo>
-      <spring_reference>0.0</spring_reference>  <!-- Neutral position -->
-      <spring_stiffness>50.0</spring_stiffness> <!-- Spring constant -->
-      <damping>0.5</damping>                   <!-- Damping coefficient -->
-    </gazebo>
   </joint>
 </xacro:macro>
@@ -242,5 +218,5 @@
         <geometry><cylinder radius="${wheel_radius}" length="${wheel_length}"/></geometry>
         <origin xyz="0 0 0" rpy="1.5707 0 0"/>
-        <material name="gray"><color rgba="${wheel_color}"/></material>
+        <material name="grey"/>
       </visual>
       <collision>
@@ -260,8 +236,4 @@
     <origin xyz="${origin_x} ${origin_y} ${origin_z}"/>
     <axis xyz="0 1 0"/> <!-- Rotate around y-axis -->
-    <gazebo>
-      <mu1>0.7</mu1> <!-- Primary friction coefficient -->
-      <mu2>0.7</mu2> <!-- Secondary friction coefficient -->
-    </gazebo>
   </joint>
 </xacro:macro>
