Commit message: Update rocker_bogie.urdf.xacro

File: src/rocker_bogie/urdf/rocker_bogie.urdf.xacro (robot description, xacro)
@@ -45,43 +45,157 @@
 </joint>
   <!-- Macro for Chassis -->
-  <xacro:macro name="chassis">
-    <link name="chassis">
-      <visual><geometry><box size="${chassis_size}"/></geometry><material name="green"><color rgba="0 1 0 1"/></material></visual>
-      <collision><geometry><box size="${chassis_size}"/></geometry></collision>
-      <inertial><mass value="5.3"/><origin xyz="0 0 0"/><inertia ixx="0.1" ixy="0" ixz="0" iyy="0.1" iyz="0" izz="0.2"/></inertial>
-    </link>
-  </xacro:macro>
+<xacro:macro name="chassis" params="">
+  <link name="chassis">
+    <visual>
+      <geometry>
+        <box size="${chassis_size}"/>
+      </geometry>
+      <origin xyz="0 0 0"/>
+      <material name="green">
+        <color rgba="0 1 0 1"/>
+      </material>
+    </visual>
+    <collision>
+      <geometry>
+        <box size="${chassis_size}"/>
+      </geometry>
+      <origin xyz="0 0 0"/>
+    </collision>
+    <inertial>
+      <mass value="5.3"/>
+      <!-- <mass value="15"/> -->
+      <origin xyz="0 0 0"/>  <!-- Set CoM to the geometric center -->
+      <inertia ixx="0.1" ixy="0" ixz="0" iyy="0.1" iyz="0" izz="0.2"/>
+    </inertial>
+  </link>
+</xacro:macro>
   <!-- Macro for Cylinder Connector -->
-  <xacro:macro name="cylinder_connector" params="name position_y">
-    <link name="${name}">
-      <visual><geometry><cylinder radius="0.0075" length="0.03"/></geometry><origin xyz="0 ${position_y} 0" rpy="1.5707 0 0"/><material name="gray"><color rgba="0.5 0.5 0.5 1"/></material></visual>
-      <collision><geometry><cylinder radius="0.0075" length="0.028"/></geometry></collision>
-      <inertial><mass value="0.5"/><origin xyz="0 ${position_y} 0"/><inertia ixx="0.00005" iyy="0.00005" izz="0.0001"/></inertial>
-    </link>
-  </xacro:macro>
+<xacro:macro name="cylinder_connector" params="name position_y">
+  <link name="${name}">
+    <visual>
+      <geometry>
+        <cylinder radius="0.0075" length="0.03"/>
+      </geometry>
+      <origin xyz="0 ${position_y} 0" rpy="1.5707 0 0"/>
+      <material name="gray">
+        <color rgba="0.5 0.5 0.5 1"/>
+      </material>
+    </visual>
+    <collision>
+      <geometry>
+        <cylinder radius="0.0075" length="0.028"/>
+      </geometry>
+      <origin xyz="0 ${position_y} 0" rpy="1.5707 0 0"/>
+    </collision>
+    <inertial>
+      <mass value="0.5"/>
+      <origin xyz="0 ${position_y} 0"/>  <!-- CoM aligned with connector -->
+      <inertia ixx="0.00005" ixy="0" ixz="0" iyy="0.00005" iyz="0" izz="0.0001"/>
+    </inertial>
+  </link>
+</xacro:macro>
   <!-- Macro for Rocker Arms -->
-  <xacro:macro name="rocker_arm" params="name position_y">
-    <link name="${name}">
-      <visual><geometry><box size="0.32 0.024 0.024"/></geometry><origin xyz="-0.147 ${position_y} 0"/><material name="blue"><color rgba="${blue_color}"/></material></visual>
-      <visual><geometry><box size="0.024 0.024 0.186"/></geometry><origin xyz="-0.294 ${position_y} -0.1"/><material name="blue"><color rgba="${blue_color}"/></material></visual>
-      <visual><geometry><box size="0.024 0.024 0.12"/></geometry><origin xyz="0.055 ${position_y} -0.055" rpy="0 -0.61 0"/><material name="blue"><color rgba="${blue_color}"/></material></visual>
-      <collision><geometry><box size="0.32 0.024 0.024"/></geometry><origin xyz="-0.147 ${position_y} 0"/></collision>
-      <collision><geometry><box size="0.024 0.024 0.186"/></geometry><origin xyz="-0.294 ${position_y} -0.1"/></collision>
-      <collision><geometry><box size="0.024 0.024 0.12"/></geometry><origin xyz="0.055 ${position_y} -0.055" rpy="0 -0.61 0"/></collision>
-      <inertial><mass value="0.25"/><origin xyz="-0.15 ${position_y} 0"/><inertia ixx="0.005" iyy="0.006" izz="0.007"/></inertial>
-    </link>
-  </xacro:macro>
+<xacro:macro name="rocker_arm" params="name position_y">
+  <link name="${name}">
+    <visual> <!-- Horizontal Bar Collision -->
+      <geometry><box size="0.32 0.024 0.024"/></geometry>
+      <origin xyz="-0.147 ${position_y} 0"/>
+      <material name="blue"><color rgba="${blue_color}"/></material>
+    </visual>
+    <visual> <!-- Vertical Bar Collision -->
+      <geometry><box size="0.024 0.024 0.186"/></geometry>
+      <origin xyz="-0.294 ${position_y} -0.1"/>
+      <material name="blue"><color rgba="${blue_color}"/></material>
+    </visual>
+    <visual> <!-- Rotating Bar Collision -->
+      <geometry><box size="0.024 0.024 0.12"/></geometry>
+      <origin xyz="0.055 ${position_y} -0.055" rpy="0 -0.61 0"/>
+      <material name="blue"><color rgba="${blue_color}"/></material>
+    </visual>
+    <collision> <!-- Horizontal Bar Collision -->
+      <geometry>
+        <box size="0.32 0.024 0.024"/>
+      </geometry>
+      <origin xyz="-0.147 ${position_y} 0"/>
+    </collision>
+    <collision> <!-- Vertical Bar Collision -->
+      <geometry>
+        <box size="0.024 0.024 0.186"/>
+      </geometry>
+      <origin xyz="-0.294 ${position_y} -0.1"/>
+    </collision>
+    <collision> <!-- Rotating Bar Collision -->
+      <geometry>
+        <box size="0.024 0.024 0.12"/>
+      </geometry>
+      <origin xyz="0.055 ${position_y} -0.055" rpy="0 -0.61 0"/>
+    </collision>
+    <inertial>
+      <!-- Adjusted mass to match the size -->
+      <mass value="0.25"/>
+      <!-- <mass value="3"/>   -->
+      <!-- CoM aligned to the center of the rocker arm -->
+      <origin xyz="-0.15 ${position_y} 0"/>
+      <!-- Adjusted inertia tensor values -->
+      <inertia ixx="0.005" ixy="0" ixz="0" iyy="0.006" iyz="0" izz="0.007"/>
+    </inertial>
+  </link>
+</xacro:macro>
   <!-- Macro for Bogie Arms -->
-  <xacro:macro name="bogie_arm" params="name position_y">
-    <link name="${name}">
-      <visual><geometry><box size="0.07 0.024 0.024"/></geometry><origin xyz="0.177 ${position_y} 0.1"/><material name="orange"><color rgba="${orange_color}"/></material></visual>
-      <visual><geometry><box size="0.024 0.024 0.162"/></geometry><origin xyz="0.2 ${position_y} 0.01"/><material name="orange"><color rgba="${orange_color}"/></material></visual>
-      <visual><geometry><box size="0.024 0.024 0.323"/></geometry><origin xyz="0.01 ${position_y} 0.01" rpy="0 0.96 0"/><material name="orange"><color rgba="${orange_color}"/></material></visual>
-      <collision><geometry><box size="0.07 0.024 0.024"/></geometry><origin xyz="0.177 ${position_y} 0.1"/></collision>
-      <collision><geometry><box size="0.024 0.024 0.162"/></geometry><origin xyz="0.2 ${position_y} 0.01"/></collision>
-      <collision><geometry><box size="0.024 0.024 0.323"/></geometry><origin xyz="0.01 ${position_y} 0.01" rpy="0 0.96 0"/></collision>
-      <inertial><mass value="0.4"/><inertia ixx="0.004" iyy="0.004" izz="0.008"/></inertial>
-    </link>
-  </xacro:macro>
+<xacro:macro name="bogie_arm" params="name position_y">
+  <link name="${name}">
+    <visual> <!-- Horizontal Bar -->
+      <geometry>
+        <box size="0.07 0.024 0.024"/>
+      </geometry>
+      <origin xyz="0.177 ${position_y} 0.1"/>
+      <material name="orange">
+        <color rgba="${orange_color}"/>
+      </material>
+    </visual>
+    <visual> <!-- Front Vertical Bar -->
+      <geometry>
+        <box size="0.024 0.024 0.162"/>
+      </geometry>
+      <origin xyz="0.2 ${position_y} 0.01"/>
+      <material name="orange">
+        <color rgba="${orange_color}"/>
+      </material>
+    </visual>
+    <visual> <!-- Back Rotating Bar -->
+      <geometry>
+        <box size="0.024 0.024 0.323"/>
+      </geometry>
+      <origin xyz="0.01 ${position_y} 0.01" rpy="0 0.96 0"/>
+      <material name="orange">
+        <color rgba="${orange_color}"/>
+      </material>
+    </visual>
+    <collision> <!-- Horizontal Bar Collision -->
+      <geometry>
+        <box size="0.07 0.024 0.024"/>
+      </geometry>
+      <origin xyz="0.177 ${position_y} 0.1"/>
+    </collision>
+    <collision> <!-- Front Vertical Bar Collision -->
+      <geometry>
+        <box size="0.024 0.024 0.162"/>
+      </geometry>
+      <origin xyz="0.2 ${position_y} 0.01"/>
+    </collision>
+    <collision> <!-- Back Rotating Bar Collision -->
+      <geometry>
+        <box size="0.024 0.024 0.323"/>
+      </geometry>
+      <origin xyz="0.01 ${position_y} 0.01" rpy="0 0.96 0"/>
+    </collision>
+    <inertial>
+      <mass value="0.4"/>
+      <!-- <mass value="2.5"/> -->
+      <origin xyz="0 0 0"/>
+      <inertia ixx="0.004" ixy="0" ixz="0" iyy="0.004" iyz="0" izz="0.008"/>
+    </inertial>
+  </link>
+</xacro:macro>
   <!-- Create Links -->
   <xacro:chassis/>
@@ -92,48 +206,69 @@
   <xacro:cylinder_connector name="cylinder_connector_left" position_y="0.145"/>
   <xacro:cylinder_connector name="cylinder_connector_right" position_y="-0.145"/>
-  <!-- MACRO: Fixed Joints -->
-  <xacro:macro name="fixed_joint" params="joint_name parent_link child_link origin_z">
-    <joint name="${joint_name}" type="fixed"><parent link="${parent_link}"/><child link="${child_link}"/><origin xyz="0 0 ${origin_z}"/></joint>
-  </xacro:macro>
+ <!-- MACRO : Fixed Joints -->
+<xacro:macro name="fixed_joint" params="joint_name parent_link child_link origin_z">
+  <joint name="${joint_name}" type="fixed">
+    <parent link="${parent_link}"/>
+    <child link="${child_link}"/>
+    <origin xyz="0 0 ${origin_z}"/>
+  </joint>
+</xacro:macro>
   <!-- Create Fixed Joints -->
-  <xacro:fixed_joint joint_name="base_to_chassis" parent_link="base_link" child_link="chassis" origin_z="0"/>
-  <xacro:fixed_joint joint_name="joint_chassis_to_cylinder_left" parent_link="chassis" child_link="cylinder_connector_left" origin_z="0"/>
-  <xacro:fixed_joint joint_name="joint_chassis_to_cylinder_right" parent_link="chassis" child_link="cylinder_connector_right" origin_z="0"/>
-  <!-- MACRO: Revolute Joints -->
-  <xacro:macro name="revolute_joint" params="joint_name parent_link child_link origin_x origin_y origin_z">
-    <joint name="${joint_name}" type="revolute">
-      <parent link="${parent_link}"/>
-      <child link="${child_link}"/>
-      <origin xyz="${origin_x} ${origin_y} ${origin_z}"/>
-      <axis xyz="0 1 0"/>
-      <limit lower="-0.26" upper="0.26" velocity="100" effort="100"/>
-      <dynamics damping="0.5" spring_stiffness="50"/>
-      <gazebo><spring_reference>0.0</spring_reference><spring_stiffness>50.0</spring_stiffness><damping>0.5</damping></gazebo>
-    </joint>
-  </xacro:macro>
-  <!-- Create Revolute Joints -->
+<xacro:fixed_joint joint_name="base_to_chassis" parent_link="base_link" child_link="chassis" origin_z="0"/>
+<xacro:fixed_joint joint_name="joint_chassis_to_cylinder_left" parent_link="chassis" child_link="cylinder_connector_left" origin_z="0"/>
+<xacro:fixed_joint joint_name="joint_chassis_to_cylinder_right" parent_link="chassis" child_link="cylinder_connector_right" origin_z="0"/>
+  <!-- MACRO : Revolute Joints -->
+<xacro:macro name="revolute_joint"
+params="joint_name parent_link child_link origin_x origin_y origin_z">
+  <joint name="${joint_name}" type="revolute">
+    <parent link="${parent_link}"/>
+    <child link="${child_link}"/>
+    <origin xyz="${origin_x} ${origin_y} ${origin_z}"/>
+    <axis xyz="0 1 0"/>
+    <limit lower="-0.26" upper="0.26" velocity="100" effort="100"/>
+    <dynamics damping="0.5" spring_stiffness="50"/>
+    <gazebo>
+      <spring_reference>0.0</spring_reference>  <!-- Neutral position -->
+      <spring_stiffness>50.0</spring_stiffness> <!-- Spring constant -->
+      <damping>0.5</damping>                   <!-- Damping coefficient -->
+    </gazebo>
+  </joint>
+</xacro:macro>
+  <!-- Create Relovute joints : CYlinder-Rocker-Bogie-->
   <xacro:revolute_joint joint_name="joint_cylinder_left_to_rocker_left" parent_link="cylinder_connector_left" child_link="rocker_left" origin_x="0" origin_y="0.165" origin_z="0"/>
   <xacro:revolute_joint joint_name="joint_cylinder_left_to_rocker_right" parent_link="cylinder_connector_right" child_link="rocker_right" origin_x="0" origin_y="-0.165" origin_z="0"/>
   <xacro:revolute_joint joint_name="joint_rocker_to_bogie_left" parent_link="rocker_left" child_link="bogie_left" origin_x="0.1" origin_y="0" origin_z="-0.1"/>
   <xacro:revolute_joint joint_name="joint_rocker_to_bogie_right" parent_link="rocker_right" child_link="bogie_right" origin_x="0.1" origin_y="0" origin_z="-0.1"/>
-  <!-- Macro: Wheels -->
+  <!-- Macro  Wheels links -->
   <xacro:macro name="wheel" params="name">
     <link name="${name}">
-      <visual><geometry><cylinder radius="${wheel_radius}" length="${wheel_length}"/></geometry><origin rpy="1.5707 0 0"/><material name="gray"><color rgba="${wheel_color}"/></material></visual>
-      <collision><geometry><cylinder radius="${wheel_radius}" length="${wheel_length}"/></geometry></collision>
-      <inertial><mass value="4"/><inertia ixx="0.0005" iyy="0.0005" izz="0.001"/></inertial>
+      <visual>
+        <geometry><cylinder radius="${wheel_radius}" length="${wheel_length}"/></geometry>
+        <origin xyz="0 0 0" rpy="1.5707 0 0"/>
+        <material name="gray"><color rgba="${wheel_color}"/></material>
+      </visual>
+      <collision>
+        <geometry><cylinder radius="${wheel_radius}" length="${wheel_length}"/></geometry>
+        <origin xyz="0 0 0" rpy="1.5707 0 0"/>
+      </collision>
+      <inertial><mass value="4"/><origin xyz="0 0 0"/>
+        <inertia ixx="0.0005" ixy="0" ixz="0" iyy="0.0005" iyz="0" izz="0.001"/>
+      </inertial>
     </link>
   </xacro:macro>
-  <!-- MACRO: Wheel Joints -->
-  <xacro:macro name="wheel_joint" params="wheel_name parent_link origin_x origin_y origin_z">
-    <joint name="joint_${wheel_name}" type="continuous">
-      <parent link="${parent_link}"/>
-      <child link="${wheel_name}"/>
-      <origin xyz="${origin_x} ${origin_y} ${origin_z}"/>
-      <axis xyz="0 1 0"/>
-      <gazebo><mu1>2.0</mu1><mu2>2.0</mu2></gazebo>
-    </joint>
-  </xacro:macro>
-  <!-- Create Wheel Links and Joints -->
+<!-- MACRO : Wheel Joints -->
+<xacro:macro name="wheel_joint" params="wheel_name parent_link origin_x origin_y origin_z">
+  <joint name="joint_${wheel_name}" type="continuous">
+    <parent link="${parent_link}"/> <!-- Attach the wheel to the correct parent link (e.g., bogie or rocker) -->
+    <child link="${wheel_name}"/>
+    <origin xyz="${origin_x} ${origin_y} ${origin_z}"/>
+    <axis xyz="0 1 0"/> <!-- Rotate around y-axis -->
+    <gazebo>
+      <mu1>2.0</mu1> <!-- Primary friction coefficient -->
+      <mu2>2.0</mu2> <!-- Secondary friction coefficient -->
+    </gazebo>
+  </joint>
+</xacro:macro>
+<!-- Create Wheel link  -->
   <xacro:wheel name="wheel_front_left"/>
   <xacro:wheel name="wheel_middle_left"/>
@@ -142,53 +277,52 @@
   <xacro:wheel name="wheel_middle_right"/>
   <xacro:wheel name="wheel_back_right"/>
-  <!-- Create Wheel Joint  -->
-  <xacro:wheel_joint wheel_name="wheel_front_left" parent_link="bogie_left" origin_x="0.2" origin_y="0.03" origin_z="-0.07"/>
-  <xacro:wheel_joint wheel_name="wheel_middle_left" parent_link="bogie_left" origin_x="-0.12" origin_y="0.03" origin_z="-0.07"/>
-  <xacro:wheel_joint wheel_name="wheel_back_left" parent_link="rocker_left" origin_x="-0.3" origin_y="0.03" origin_z="-0.17"/>
-  <xacro:wheel_joint wheel_name="wheel_front_right" parent_link="bogie_right" origin_x="0.2" origin_y="-0.03" origin_z="-0.07"/>
-  <xacro:wheel_joint wheel_name="wheel_middle_right" parent_link="bogie_right" origin_x="-0.12" origin_y="-0.03" origin_z="-0.07"/>
-  <xacro:wheel_joint wheel_name="wheel_back_right" parent_link="rocker_right" origin_x="-0.3" origin_y="-0.03" origin_z="-0.17"/>
-  <gazebo reference="lidar_link">
-    <material name="black"><color rgba="0.0 0.0 0.0 1.0"/></material>
-    <sensor type="ray" name="lidar_sensor">
-      <pose>0 0 0.3 0 0 0</pose>
-      <visualize>true</visualize>
-      <update_rate>5</update_rate>
-      <ray>
-        <scan>
-          <horizontal>
-            <samples>360</samples>
-            <resolution>1</resolution>
-            <min_angle>0</min_angle> <!-- -90 degrees -->
-            <max_angle>6.28</max_angle>  <!-- +90 degrees -->
-          </horizontal>
-        </scan>
-        <range>
-          <min>0.2</min> <!-- Min detection distance -->
-          <max>3.5</max> <!-- Max detection distance -->
-          <resolution>0.015</resolution>
-        </range>
-        <noise>
-          <type>gaussian</type>
-          <mean>0.0</mean>
-          <stddev>0.01</stddev>
-        </noise>
-      </ray>
-      <plugin name="gazebo_ros_laser" filename="libgazebo_ros_laser.so">
-        <topicName>scan</topicName>
-        <frameName>lidar_link</frameName>
-      </plugin>
-    </sensor>
-  </gazebo>
-  <!-- Skid Steering Plugin -->
-  <gazebo>
-    <plugin name="skid_steering_plugin" filename="libskid_steering_plugin.so">
-      <left_joint>joint_wheel_front_left</left_joint>
-      <left_joint>joint_wheel_middle_left</left_joint>
-      <left_joint>joint_wheel_back_left</left_joint>
-      <right_joint>joint_wheel_front_right</right_joint>
-      <right_joint>joint_wheel_middle_right</right_joint>
-      <right_joint>joint_wheel_back_right</right_joint>
+<!-- Create Wheel Joint  -->
+<xacro:wheel_joint wheel_name="wheel_front_left" parent_link="bogie_left" origin_x="0.2" origin_y="0.03" origin_z="-0.07"/>
+<xacro:wheel_joint wheel_name="wheel_middle_left" parent_link="bogie_left" origin_x="-0.12" origin_y="0.03" origin_z="-0.07"/>
+<xacro:wheel_joint wheel_name="wheel_back_left" parent_link="rocker_left" origin_x="-0.3" origin_y="0.03" origin_z="-0.17"/>
+<xacro:wheel_joint wheel_name="wheel_front_right" parent_link="bogie_right" origin_x="0.2" origin_y="-0.03" origin_z="-0.07"/>
+<xacro:wheel_joint wheel_name="wheel_middle_right" parent_link="bogie_right" origin_x="-0.12" origin_y="-0.03" origin_z="-0.07"/>
+<xacro:wheel_joint wheel_name="wheel_back_right" parent_link="rocker_right" origin_x="-0.3" origin_y="-0.03" origin_z="-0.17"/>
+<gazebo reference="lidar_link">
+  <material name="black"><color rgba="0.0 0.0 0.0 1.0"/></material>
+  <sensor type="ray" name="lidar_sensor">
+    <pose>0 0 0.3 0 0 0</pose>
+    <visualize>true</visualize>
+    <update_rate>5</update_rate>
+    <ray>
+      <scan>
+        <horizontal>
+          <samples>360</samples>
+          <resolution>1</resolution>
+          <min_angle>0</min_angle> <!-- -90 degrees -->
+          <max_angle>6.28</max_angle>  <!-- +90 degrees -->
+        </horizontal>
+      </scan>
+      <range>
+        <min>0.2</min> <!-- Min detection distance -->
+        <max>3.5</max> <!-- Max detection distance -->
+        <resolution>0.015</resolution>
+      </range>
+      <noise>
+        <type>gaussian</type>
+        <mean>0.0</mean>
+        <stddev>0.01</stddev>
+      </noise>
+    </ray>
+    <plugin name="gazebo_ros_laser" filename="libgazebo_ros_laser.so">
+      <topicName>scan</topicName>
+      <frameName>lidar_link</frameName>
     </plugin>
-  </gazebo>
+  </sensor>
+</gazebo>
+<gazebo>
+  <plugin name="skid_steering_plugin" filename="libskid_steering_plugin.so">
+    <left_joint>joint_wheel_front_left</left_joint>
+    <left_joint>joint_wheel_middle_left</left_joint>
+    <left_joint>joint_wheel_back_left</left_joint>
+    <right_joint>joint_wheel_front_right</right_joint>
+    <right_joint>joint_wheel_middle_right</right_joint>
+    <right_joint>joint_wheel_back_right</right_joint>
+  </plugin>
+</gazebo>
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
Commit message: SLAM

File: src/rocker_bogie/urdf/rocker_bogie.urdf.xacro (robot description, xacro)
@@ -10,4 +10,8 @@
 <!-- Base Link at the Center of the Chassis -->
 <link name="base_link">
+  <!-- <inertial>
+    <mass value="0.1"/>
+    <inertia ixx="0.001" ixy="0" ixz="0" iyy="0.001" iyz="0" izz="0.001"/>
+  </inertial> -->
   <visual>
     <geometry>
@@ -29,13 +33,13 @@
       </material>
   </visual>
-  <collision>
+  <!-- <collision>
       <geometry>
           <cylinder length="0.05" radius="0.02"/>
       </geometry>
-  </collision>
-  <inertial>
-      <mass value="0.1"/> <!-- Adjust mass -->
+  </collision> -->
+  <!-- <inertial>
+      <mass value="0.1"/>
       <inertia ixx="0.01" ixy="0.0" ixz="0.0" iyy="0.01" iyz="0.0" izz="0.01"/>
-  </inertial>
+  </inertial> -->
 </link>
 <joint name="lidar_joint" type="fixed">
@@ -66,5 +70,5 @@
       <!-- <mass value="15"/> -->
       <origin xyz="0 0 0"/>  <!-- Set CoM to the geometric center -->
-      <inertia ixx="0.1" ixy="0" ixz="0" iyy="0.1" iyz="0" izz="0.2"/>
+      <inertia ixx="0.5" ixy="0" ixz="0" iyy="0.5" iyz="0" izz="0.8"/>
     </inertial>
   </link>
@@ -287,5 +291,6 @@
   <material name="black"><color rgba="0.0 0.0 0.0 1.0"/></material>
   <sensor type="ray" name="lidar_sensor">
-    <pose>0 0 0.3 0 0 0</pose>
+    <!-- <pose>0 0 0.3 0 0 0</pose> -->
+    <origin xyz="0 0 0.3" rpy="0 0 0"/>
     <visualize>true</visualize>
     <update_rate>5</update_rate>
@@ -326,3 +331,6 @@
   </plugin>
 </gazebo>
+<!-- <gazebo>
+  <plugin name="odometry_plugin" filename="libodometry_plugin.so"/>
+</gazebo> -->
 </robot>

Commit message: urdf

File: src/rocker_bogie/urdf/rocker_bogie.urdf.xacro (robot description, xacro)
@@ -29,7 +29,7 @@
           <cylinder length="0.05" radius="0.02"/> <!-- Adjust dimensions as needed -->
       </geometry>
-      <material name="green_material">
-          <color rgba="0.0 1.0 0.0 0.5"/> <!-- Semi-transparent green for visualization -->
-      </material>
+    <!--  <material name="green_material">
+        <color rgba="0.0 1.0 0.0 0.5"/>
+    </material> -->
   </visual>
   <!-- <collision>
@@ -46,5 +46,5 @@
   <parent link="base_link"/>
   <child link="lidar_link"/>
-  <origin xyz="0 0 0.3" rpy="0 0 0"/> <!-- Position the LiDAR slightly above the rover chassis -->
+  <origin xyz="0 0 0.2" rpy="0 0 0"/> <!-- Position the LiDAR slightly above the rover chassis -->
 </joint>
   <!-- Macro for Chassis -->
@@ -292,7 +292,7 @@
   <sensor type="ray" name="lidar_sensor">
     <!-- <pose>0 0 0.3 0 0 0</pose> -->
-    <origin xyz="0 0 0.3" rpy="0 0 0"/>
+    <origin xyz="0 0 0.2" rpy="0 0 0"/>
     <visualize>true</visualize>
-    <update_rate>5</update_rate>
+    <update_rate>20</update_rate>
     <ray>
       <scan>

Commit message: urdf

File: src/rocker_bogie/urdf/rocker_bogie.urdf.xacro (robot description, xacro)
@@ -29,17 +29,5 @@
           <cylinder length="0.05" radius="0.02"/> <!-- Adjust dimensions as needed -->
       </geometry>
-    <!--  <material name="green_material">
-        <color rgba="0.0 1.0 0.0 0.5"/>
-    </material> -->
   </visual>
-  <!-- <collision>
-      <geometry>
-          <cylinder length="0.05" radius="0.02"/>
-      </geometry>
-  </collision> -->
-  <!-- <inertial>
-      <mass value="0.1"/>
-      <inertia ixx="0.01" ixy="0.0" ixz="0.0" iyy="0.01" iyz="0.0" izz="0.01"/>
-  </inertial> -->
 </link>
 <joint name="lidar_joint" type="fixed">
