Commit message: urdf

File: src/rocker_bogie/urdf/rocker_bogie.urdf.xacro (robot description, xacro)
@@ -10,8 +10,4 @@
 <!-- Base Link at the Center of the Chassis -->
 <link name="base_link">
-  <!-- <inertial>
-    <mass value="0.1"/>
-    <inertia ixx="0.001" ixy="0" ixz="0" iyy="0.001" iyz="0" izz="0.001"/>
-  </inertial> -->
   <visual>
     <geometry>

Commit message: separate plugin

File: src/rocker_bogie/urdf/rocker_bogie.urdf.xacro (robot description, xacro)
@@ -1,4 +1,5 @@
 <?xml version="1.0"?>
 <robot xmlns:xacro="http://www.ros.org/wiki/xacro" name="rocker_bogie">
+  <xacro:include filename="$(find rocker_bogie)/urdf/plugins.xacro"/>
   <!-- Properties for reuse -->
   <xacro:property name="wheel_radius" value="0.07"/>
@@ -22,7 +23,8 @@
 <link name="lidar_link">
   <visual>
+    <origin xyz="0 0 0.1" rpy="0 0 0" />
     <geometry>
-          <cylinder length="0.05" radius="0.02"/> <!-- Adjust dimensions as needed -->
-      </geometry>
+      <cylinder length="0.05" radius="0.02"/>
+    </geometry>
   </visual>
 </link>
@@ -31,4 +33,10 @@
   <child link="lidar_link"/>
   <origin xyz="0 0 0.2" rpy="0 0 0"/> <!-- Position the LiDAR slightly above the rover chassis -->
+</joint>
+<link name="base_footprint"/>
+<joint name="base_footprint_joint" type="fixed">
+    <parent link="base_footprint"/>
+    <child link="base_link"/>
+    <origin xyz="0 0 -0.05" rpy="0 0 0"/>
 </joint>
   <!-- Macro for Chassis -->
@@ -272,49 +280,3 @@
 <xacro:wheel_joint wheel_name="wheel_middle_right" parent_link="bogie_right" origin_x="-0.12" origin_y="-0.03" origin_z="-0.07"/>
 <xacro:wheel_joint wheel_name="wheel_back_right" parent_link="rocker_right" origin_x="-0.3" origin_y="-0.03" origin_z="-0.17"/>
-<gazebo reference="lidar_link">
-  <material name="black"><color rgba="0.0 0.0 0.0 1.0"/></material>
-  <sensor type="ray" name="lidar_sensor">
-    <!-- <pose>0 0 0.3 0 0 0</pose> -->
-    <origin xyz="0 0 0.2" rpy="0 0 0"/>
-    <visualize>true</visualize>
-    <update_rate>20</update_rate>
-    <ray>
-      <scan>
-        <horizontal>
-          <samples>360</samples>
-          <resolution>1</resolution>
-          <min_angle>0</min_angle> <!-- -90 degrees -->
-          <max_angle>6.28</max_angle>  <!-- +90 degrees -->
-        </horizontal>
-      </scan>
-      <range>
-        <min>0.2</min> <!-- Min detection distance -->
-        <max>3.5</max> <!-- Max detection distance -->
-        <resolution>0.015</resolution>
-      </range>
-      <noise>
-        <type>gaussian</type>
-        <mean>0.0</mean>
-        <stddev>0.01</stddev>
-      </noise>
-    </ray>
-    <plugin name="gazebo_ros_laser" filename="libgazebo_ros_laser.so">
-      <topicName>scan</topicName>
-      <frameName>lidar_link</frameName>
-    </plugin>
-  </sensor>
-</gazebo>
-<gazebo>
-  <plugin name="skid_steering_plugin" filename="libskid_steering_plugin.so">
-    <left_joint>joint_wheel_front_left</left_joint>
-    <left_joint>joint_wheel_middle_left</left_joint>
-    <left_joint>joint_wheel_back_left</left_joint>
-    <right_joint>joint_wheel_front_right</right_joint>
-    <right_joint>joint_wheel_middle_right</right_joint>
-    <right_joint>joint_wheel_back_right</right_joint>
-  </plugin>
-</gazebo>
-<!-- <gazebo>
-  <plugin name="odometry_plugin" filename="libodometry_plugin.so"/>
-</gazebo> -->
 </robot>

Commit message: adjust inertia

File: src/rocker_bogie/urdf/rocker_bogie.urdf.xacro (robot description, xacro)
@@ -49,5 +49,5 @@
         <!-- <mass value="15"/> -->
         <origin xyz="0 0 0" />
-        <inertia ixx="0.5" ixy="0" ixz="0" iyy="0.5" iyz="0" izz="0.8" />
+        <inertia ixx="0.033" ixy="0" ixz="0" iyy="0.052" iyz="0" izz="0.073" />
       </inertial>
     </link>
@@ -210,19 +210,15 @@
       <origin xyz="${origin_x} ${origin_y} ${origin_z}" />
       <axis xyz="0 1 0" />
-      <limit lower="-0.26" upper="0.26" velocity="100" effort="100" />
-      <dynamics damping="0.5" spring_stiffness="50" />
+      <limit lower="-0.33" upper="0.33" velocity="100" effort="50" />
+      <dynamics damping="1" spring_stiffness="100" />
     </joint>
   </xacro:macro>
   <!-- Create Relovute joints : CYlinder-Rocker-Bogie-->
   <xacro:revolute_joint joint_name="joint_cylinder_left_to_rocker_left"
-    parent_link="cylinder_connector_left" child_link="rocker_left" origin_x="0" origin_y="0.165"
-    origin_z="0" />
+    parent_link="cylinder_connector_left" child_link="rocker_left" origin_x="0" origin_y="0.165" origin_z="0" />
   <xacro:revolute_joint joint_name="joint_cylinder_left_to_rocker_right"
-    parent_link="cylinder_connector_right" child_link="rocker_right" origin_x="0" origin_y="-0.165"
-    origin_z="0" />
-  <xacro:revolute_joint joint_name="joint_rocker_to_bogie_left" parent_link="rocker_left"
-    child_link="bogie_left" origin_x="0.1" origin_y="0" origin_z="-0.1" />
-  <xacro:revolute_joint joint_name="joint_rocker_to_bogie_right" parent_link="rocker_right"
-    child_link="bogie_right" origin_x="0.1" origin_y="0" origin_z="-0.1" />
+    parent_link="cylinder_connector_right" child_link="rocker_right" origin_x="0" origin_y="-0.165" origin_z="0" />
+  <xacro:revolute_joint joint_name="joint_rocker_to_bogie_left" parent_link="rocker_left" child_link="bogie_left" origin_x="0.1" origin_y="0" origin_z="-0.1" />
+  <xacro:revolute_joint joint_name="joint_rocker_to_bogie_right" parent_link="rocker_right" child_link="bogie_right" origin_x="0.1" origin_y="0" origin_z="-0.1" />
   <!-- Macro  Wheels links -->
   <xacro:macro name="wheel" params="name">

Commit message: urdf

File: src/rocker_bogie/urdf/rocker_bogie.urdf.xacro (robot description, xacro)
@@ -46,6 +46,5 @@
       </collision>
       <inertial>
-        <mass value="5.3" />
-        <!-- <mass value="15"/> -->
+        <mass value="6.3" />
         <origin xyz="0 0 0" />
         <inertia ixx="0.033" ixy="0" ixz="0" iyy="0.052" iyz="0" izz="0.073" />
@@ -172,7 +171,7 @@
       </collision>
       <inertial>
-        <mass value="0.4" />
+        <mass value="0.2" />
         <!-- <mass value="2.5"/> -->
-        <origin xyz="0 0 0" />
+        <origin xyz="0.086 ${position_y} 0" />
         <inertia ixx="0.004" ixy="0" ixz="0" iyy="0.004" iyz="0" izz="0.008" />
       </inertial>
