Commit message: urdf no lidar

File: src/rocker_bogie/urdf/rocker_bogie.urdf_no_lidar.xacro (robot description, xacro)
@@ -171,7 +171,7 @@
       </collision>
       <inertial>
-        <mass value="0.4" />
+        <mass value="0.2" />
         <!-- <mass value="2.5"/> -->
-        <origin xyz="0 0 0" />
+        <origin xyz="0.086 ${position_y} 0" />
         <inertia ixx="0.004" ixy="0" ixz="0" iyy="0.004" iyz="0" izz="0.008" />
       </inertial>
